Commit message: added two new scripts, script one is newScanner which scans the area around the rover using a laser and automove is to use this data to try to move around..Modified the plugin and launch files to have the sensor.. also added hokuyo lidar scanner before the built in scanner and then discarded it

File: urdf/rover.urdf.xacro (robot description, xacro)
@@ -1,4 +1,4 @@
 <?xml version="1.0"?>
-<robot xmlns:xacro = "http://www.ros.org/wiki/xacro" name="rover">
+<robot xmlns:xacro="http://www.ros.org/wiki/xacro" name="rover">
   <xacro:property name="base_width" value="0.16"/>
   <xacro:property name="base_len" value="0.16"/>
@@ -7,5 +7,8 @@
   <xacro:property name="wheel_separation" value="0.15"/>
   <xacro:property name="wheel_joint_offset" value="0.02"/>
-  <xacro:include filename="$(find rover)/urdf/rover_gazebo_plugins.xacro"/>
+  <xacro:property name="caster_wheel_radius" value="${wheel_radius/2}"/>
+  <xacro:property name="caster_wheel_mass" value="0.001"/>
+  <xacro:property name="caster_wheel_joint_offset" value="-0.052"/>
+  <!--Color Properties-->
   <material name="blue">
     <color rgba="0 0 0.8 1"/>
@@ -20,5 +23,12 @@
     <color rgba="0.8 0.0 0.0 1.0"/>
   </material>
-   <xacro:macro name="box_inertia" params="m w h d">
+  <!--Interial macros-->
+  <xacro:macro name="cylinder_inertia" params="m r h">
+    <inertial>
+      <mass value="${m}"/>
+      <inertia ixx="${m*(3*r*r+h*h)/12}" ixy = "0" ixz = "0" iyy="${m*(3*r*r+h*h)/12}" iyz = "0" izz="${m*r*r/2}"/>
+    </inertial>
+  </xacro:macro>
+  <xacro:macro name="box_inertia" params="m w h d">
     <inertial>
       <mass value="${m}"/>
@@ -26,6 +36,13 @@
     </inertial>
   </xacro:macro>
+  <xacro:macro name="sphere_inertia" params="m r">
+    <inertial>
+      <mass value="${m}"/>
+      <inertia ixx="${2.0*m*(r*r)/5.0}" ixy="0.0" ixz="0.0" iyy="${2.0*m*(r*r)/5.0}" iyz="0.0" izz="${2.0*m*(r*r)/5.0}"/>
+    </inertial>
+  </xacro:macro>
+  <!--Base Footprint-->
   <link name="base_footprint">
-    <xacro:box_inertia m="20" w="0.001" h="0.001" d="0.001"/>
+    <xacro:box_inertia m="10" w="0.001" h="0.001" d="0.001"/>
     <visual>
         <origin xyz="0 0 0" rpy="0 0 0" />
@@ -35,4 +52,5 @@
     </visual>
   </link>
+  <!--Base link-->
   <link name="base_link">
     <xacro:box_inertia m="10" w="${base_len}" h="${base_width}" d="0.01"/>
@@ -41,4 +59,5 @@
         <box size="${base_len} ${base_width} 0.01"/>
       </geometry>
+      <material name="black"/>
     </visual>
     <collision>
@@ -48,4 +67,5 @@
     </collision>
   </link>
+  <!--base_link to base_footprint Joint-->
   <joint name="base_link_joint" type="fixed">
     <origin xyz="0 0 ${wheel_radius + 0.005}" rpy="0 0 0" />
@@ -53,10 +73,5 @@
     <child link="base_link" />
   </joint>
-  <xacro:macro name="cylinder_inertia" params="m r h">
-    <inertial>
-      <mass value="${m}"/>
-      <inertia ixx="${m*(3*r*r+h*h)/12}" ixy = "0" ixz = "0" iyy="${m*(3*r*r+h*h)/12}" iyz = "0" izz="${m*r*r/2}"/>
-    </inertial>
-  </xacro:macro>
+  <!--Wheel link & joint macro-->
   <xacro:macro name="wheel" params="prefix reflect">
     <link name="${prefix}_wheel">
@@ -83,5 +98,83 @@
     </joint>
   </xacro:macro>
+  <!--Create Left & Right Wheel links/joints-->
   <xacro:wheel prefix="left" reflect="1"/>
   <xacro:wheel prefix="right" reflect="-1"/>
+  <!--Caster Wheel Link-->
+  <link name="caster_wheel">
+    <visual>
+      <origin xyz="0 0 0" rpy="0 0 0"/>
+      <geometry>
+        <sphere radius="${caster_wheel_radius}"/>
+      </geometry>
+      <material name="blue"/>
+    </visual>
+    <collision>
+      <origin xyz="0 0 0" rpy="0 0 0"/>
+      <geometry>
+        <sphere radius="${caster_wheel_radius}"/>
+      </geometry>
+    </collision>
+    <xacro:sphere_inertia m="10" r="${caster_wheel_radius}"/>
+  </link>
+  <!--Caster Wheel Joint-->
+  <joint name="caster_wheel_joint" type="continuous">
+    <axis xyz="0 1 0" rpy="0 0 0" />
+    <parent link="base_link"/>
+    <child link="caster_wheel"/>
+    <origin xyz="${caster_wheel_joint_offset} 0 -${caster_wheel_radius+0.005}" rpy="0 0 0"/>
+  </joint>
+<!-- laser -->
+<link name="laser">
+  <xacro:cylinder_inertia m="5" r="0.025" h="0.025"/>
+  <visual>
+    <geometry>
+      <cylinder radius="0.025" length="0.025"/>
+     </geometry>
+  </visual>
+  <collision>
+    <origin/>
+    <geometry>
+      <cylinder radius="0.025" length="0.025"/>
+    </geometry>
+  </collision>
+</link>
+<joint name="laser_joint" type="fixed">
+  <origin xyz="0 0.0 0.015" rpy="0.0 0.0 3.14"/>
+  <axis xyz="0 0 1" />
+  <parent link="base_link"/>
+  <child link="laser"/>
+</joint>
+<gazebo reference="laser">
+  <sensor type="ray" name="laser">
+      <pose>0 0 0 0 0 0</pose>
+      <visualize>false</visualize>
+      <update_rate>40</update_rate>
+      <ray>
+          <scan>
+              <horizontal>
+                  <samples>1440</samples>
+                  <resolution>0.5</resolution>
+                  <min_angle>-1.578</min_angle>
+                  <max_angle>1.578</max_angle>
+              </horizontal>
+          </scan>
+          <range>
+            <min>0.10</min>
+            <max>3.0</max>
+            <resolution>0.01</resolution>
+          </range>
+          <noise>
+            <type>gaussian</type>
+            <mean>0.0</mean>
+            <stddev>0.01</stddev>
+          </noise>
+      </ray>
+      <plugin name="laser_controller" filename="libgazebo_ros_laser.so">
+          <topicName>/scan</topicName>
+          <frameName>laser</frameName>
+      </plugin>
+  </sensor>
+</gazebo>
+  <xacro:include filename="$(find pde4430_ex2)/urdf/rover_gazebo_plugins.xacro"/>
 </robot>

File: urdf/rover_gazebo_plugins.xacro (robot description, xacro)
@@ -12,5 +12,5 @@
       <torque>20</torque>
       <commandTopic>/rover/base_controller/cmd_vel</commandTopic>
-      <odometryTopic>/rover/base_controller/odom</odometryTopic>
+      <odometryTopic>/odom</odometryTopic>
       <odometryFrame>odom</odometryFrame>
       <robotBaseFrame>base_footprint</robotBaseFrame>
